File: 5431-ButtonBoardButBetter/5431-ButtonBoardButBetter.kicad_sch (KiCad schematic)
At the start: 17 parts, among them SW1 SW_DIP_x01, SW10 SW_DIP_x01, SW11 SW_DIP_x01, SW12 SW_DIP_x01, SW13 SW_DIP_x01, SW14 SW_DIP_x01, SW15 SW_DIP_x01, SW16 SW_DIP_x01, SW2 SW_DIP_x01, SW3 SW_DIP_x01, SW4 SW_DIP_x01, SW5 SW_DIP_x01, SW6 SW_DIP_x01, SW7 SW_DIP_x01, SW8 SW_DIP_x01, SW9 SW_DIP_x01, U1 Pico

Commit message: footprints plus basic pcb setup
done
Parts:
- SW1, SW10, SW11, SW12, SW13, SW14, SW15, SW16, SW2, SW3, SW5, SW6, SW7, SW8, SW9: footprint (none) -> Button_Switch_Keyboard:SW_Cherry_MX_1.00u_PCB
Other:
- moved on the sheet: SW1, SW10, SW11, SW12, SW13, SW14, SW15, SW16, SW2, SW3, SW4, SW5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

Commit message: Updated sch
Parts:
- added SW17: SW_DIP_x01, Button_Switch_THT:SW_PUSH_6mm, symbol Switch:SW_DIP_x01
Connections:
- net GND: now also SW17.1
- net Reset: now also SW17.2
- net Sw10: now also U1.27 (GPIO21); no longer U1.12 (GPIO9)
- net Sw11: now also U1.26 (GPIO20); no longer U1.14 (GPIO10)
- net Sw12: now also U1.25 (GPIO19); no longer U1.15 (GPIO11)
- net Sw13: now also U1.24 (GPIO18); no longer U1.16 (GPIO12)
- net Sw14: now also U1.22 (GPIO17); no longer U1.17 (GPIO13)
- net Sw15: now also U1.21 (GPIO16)
- net Sw16: now also U1.20 (GPIO15)
- net Sw9: now also U1.29 (GPIO22); no longer U1.11 (GPIO8)
Other:
- moved on the sheet: U1

Commit message: added slider
Parts:
- added RV1, RV2: R_Potentiometer_US, Potentiometer_THT:Potentiometer_Bourns_PTA4543_Single_Slide, symbol Device:R_Potentiometer_US
- added U2: MCP3008, symbol Analog_ADC:MCP3008
Connections:
- net GND: now also RV1.3, RV2.3
- net +3V3: now reaches U1.36 (3V3)
- net +3V3: now also RV1.1, RV2.1
- new net: RV2.2, U2.2 (CH1)
- new net: RV1.2, U2.1 (CH0)
Changed lines of the file:
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@@
+    (stroke (width 0) (type default))
+  )
+  (wire (pts (xy 55.88 24.13) (xy 109.22 24.13))
     (stroke (width 0) (type default))
   )
@@
   )
   (wire (pts (xy 63.5 58.42) (xy 72.39 58.42))
+    (stroke (width 0) (type default))
+  )
+  (wire (pts (xy 55.88 26.67) (xy 55.88 24.13))
+    (stroke (width 0) (type default))
+  )
+  (wire (pts (xy 81.28 26.67) (xy 109.22 26.67))
     (stroke (width 0) (type default))
   )
@@
     (property "Intersheetrefs" "${INTERSHEET_REFS}" (at 192.7103 63.119 0)
       (effects (font (size 1.27 1.27)) (justify left) hide)
+    )
+  )
+  (symbol (lib_id "Device:R_Potentiometer_US") (at 81.28 30.48 90) (unit 1)
+    (in_bom yes) (on_board yes) (dnp no) (fields_autoplaced)
+    (property "Reference" "RV2" (at 81.28 34.29 90)
+      (effects (font (size 1.27 1.27)))
+    )
+    (property "Value" "R_Potentiometer_US" (at 81.28 36.83 90)
+      (effects (font (size 1.27 1.27)))
+    )
+    (property "Footprint" "Potentiometer_THT:Potentiometer_Bourns_PTA4543_Single_Slide" (at 81.28 30.48 0)
+      (effects (font (size 1.27 1.27)) hide)
+    )
+    (property "Datasheet" "~" (at 81.28 30.48 0)
+      (effects (font (size 1.27 1.27)) hide)
+    )
+    (pin "1")
+    (pin "2")
+    (pin "3")
+    (instances
+      (project "5431-ButtonBoardButBetter"
+        (path "/85ad268b-acfd-4dd1-a78b-2229ab217983"
+          (reference "RV2") (unit 1)
+        )
+      )
     )
   )
@@
     )
   )
+  (symbol (lib_id "power:+3V3") (at 107.95 60.96 270) (unit 1)
+    (in_bom yes) (on_board yes) (dnp no) (fields_autoplaced)
+    (property "Reference" "#PWR021" (at 104.14 60.96 0)
+      (effects (font (size 1.27 1.27)) hide)
+    )
+    (property "Value" "+3V3" (at 111.76 61.595 90)
+      (effects (font (size 1.27 1.27)) (justify left))
+    )
+    (property "Footprint" "" (at 107.95 60.96 0)
+      (effects (font (size 1.27 1.27)) hide)
+    )
+    (property "Datasheet" "" (at 107.95 60.96 0)
+      (effects (font (size 1.27 1.27)) hide)
+    )
+    (pin "1")
+    (instances
+      (project "5431-ButtonBoardButBetter"
+        (path "/85ad268b-acfd-4dd1-a78b-2229ab217983"
+          (reference "#PWR021") (unit 1)
+        )
+      )
+    )
+  )
   (symbol (lib_id "Switch:SW_DIP_x01") (at 177.8 91.059 0) (unit 1)
     (in_bom yes) (on_board yes) (dnp no) (fields_autoplaced)
@@
         (path "/85ad268b-acfd-4dd1-a78b-2229ab217983"
           (reference "SW11") (unit 1)
+        )
+      )
+    )
+  )
+  (symbol (lib_id "power:+3V3") (at 77.47 30.48 90) (mirror x) (unit 1)
+    (in_bom yes) (on_board yes) (dnp no)
+    (property "Reference" "#PWR022" (at 81.28 30.48 0)
+      (effects (font (size 1.27 1.27)) hide)
+    )
+    (property "Value" "+3V3" (at 73.66 31.115 90)
+      (effects (font (size 1.27 1.27)) (justify left))
+    )
+    (property "Footprint" "" (at 77.47 30.48 0)
+      (effects (font (size 1.27 1.27)) hide)
+    )
+    (property "Datasheet" "" (at 77.47 30.48 0)
+      (effects (font (size 1.27 1.27)) hide)
+    )
+    (pin "1")
+    (instances
+      (project "5431-ButtonBoardButBetter"
+        (path "/85ad268b-acfd-4dd1-a78b-2229ab217983"
+          (reference "#PWR022") (unit 1)
         )
       )
@@
         (path "/85ad268b-acfd-4dd1-a78b-2229ab217983"
           (reference "SW17") (unit 1)
+        )
+      )
+    )
+  )
+  (symbol (lib_id "power:GND") (at 85.09 30.48 90) (unit 1)
+    (in_bom yes) (on_board yes) (dnp no) (fields_autoplaced)
+    (property "Reference" "#PWR029" (at 91.44 30.48 0)
+      (effects (font (size 1.27 1.27)) hide)
+    )
+    (property "Value" "GND" (at 88.265 31.115 90)
+      (effects (font (size 1.27 1.27)) (justify right))
+    )
+    (property "Footprint" "" (at 85.09 30.48 0)
+      (effects (font (size 1.27 1.27)) hide)
+    )
+    (property "Datasheet" "" (at 85.09 30.48 0)
+      (effects (font (size 1.27 1.27)) hide)
+    )
+    (pin "1")
+    (instances
+      (project "5431-ButtonBoardButBetter"
+        (path "/85ad268b-acfd-4dd1-a78b-2229ab217983"
+          (reference "#PWR029") (unit 1)
         )
       )
@@
     )
   )
+  (symbol (lib_id "Analog_ADC:MCP3008") (at 124.46 31.75 0) (unit 1)
+    (in_bom yes) (on_board yes) (dnp no) (fields_autoplaced)
+    (property "Reference" "U2" (at 131.4959 17.78 0)
+      (effects (font (size 1.27 1.27)) (justify left))
+    )
+    (property "Value" "MCP3008" (at 131.4959 20.32 0)
+      (effects (font (size 1.27 1.27)) (justify left))
+    )
+    (property "Footprint" "" (at 127 29.21 0)
+      (effects (font (size 1.27 1.27)) hide)
+    )
+    (property "Datasheet" "http://ww1.microchip.com/downloads/en/DeviceDoc/21295d.pdf" (at 127 29.21 0)
+      (effects (font (size 1.27 1.27)) hide)
+    )
+    (pin "1")
+    (pin "10")
+    (pin "11")
+    (pin "12")
+    (pin "13")
+    (pin "14")
+    (pin "15")
+    (pin "16")
+    (pin "2")
+    (pin "3")
+    (pin "4")
+    (pin "5")
+    (pin "6")
+    (pin "7")
+    (pin "8")
+    (pin "9")
+    (instances
+      (project "5431-ButtonBoardButBetter"
+        (path "/85ad268b-acfd-4dd1-a78b-2229ab217983"
+          (reference "U2") (unit 1)
+        )
+      )
+    )
+  )
   (symbol (lib_id "power:GND") (at 112.395 93.98 90) (unit 1)
     (in_bom yes) (on_board yes) (dnp no) (fields_autoplaced)
@@
     )
   )
+  (symbol (lib_id "power:+3V3") (at 52.07 30.48 90) (mirror x) (unit 1)
+    (in_bom yes) (on_board yes) (dnp no)
+    (property "Reference" "#PWR028" (at 55.88 30.48 0)
+      (effects (font (size 1.27 1.27)) hide)
+    )
+    (property "Value" "+3V3" (at 48.26 31.115 90)
+      (effects (font (size 1.27 1.27)) (justify left))
+    )
+    (property "Footprint" "" (at 52.07 30.48 0)
+      (effects (font (size 1.27 1.27)) hide)
+    )
+    (property "Datasheet" "" (at 52.07 30.48 0)
+      (effects (font (size 1.27 1.27)) hide)
+    )
+    (pin "1")
+    (instances
+      (project "5431-ButtonBoardButBetter"
+        (path "/85ad268b-acfd-4dd1-a78b-2229ab217983"
+          (reference "#PWR028") (unit 1)
+        )
+      )
+    )
+  )
   (symbol (lib_id "power:GND") (at 67.31 68.58 270) (unit 1)
     (in_bom yes) (on_board yes) (dnp no) (fields_autoplaced)
@@
     )
   )
+  (symbol (lib_id "power:GND") (at 59.69 30.48 90) (unit 1)
+    (in_bom yes) (on_board yes) (dnp no) (fields_autoplaced)
+    (property "Reference" "#PWR030" (at 66.04 30.48 0)
+      (effects (font (size 1.27 1.27)) hide)
+    )
+    (property "Value" "GND" (at 62.865 31.115 90)
+      (effects (font (size 1.27 1.27)) (justify right))
+    )
+    (property "Footprint" "" (at 59.69 30.48 0)
+      (effects (font (size 1.27 1.27)) hide)
+    )
+    (property "Datasheet" "" (at 59.69 30.48 0)
+      (effects (font (size 1.27 1.27)) hide)
+    )
+    (pin "1")
+    (instances
+      (project "5431-ButtonBoardButBetter"
+        (path "/85ad268b-acfd-4dd1-a78b-2229ab217983"
+          (reference "#PWR030") (unit 1)
+        )
+      )
+    )
+  )
   (symbol (lib_id "power:GND") (at 139.7 125.73 0) (unit 1)
     (in_bom yes) (on_board yes) (dnp no) (fields_autoplaced)
@@
         )
       )
+    )
+  )
+  (symbol (lib_id "Device:R_Potentiometer_US") (at 55.88 30.48 90) (unit 1)
+    (in_bom yes) (on_board yes) (dnp no) (fields_autoplaced)
+    (property "Reference" "RV1" (at 55.88 34.29 90)
+      (effects (font (size 1.27 1.27)))
+    )
+    (property "Value" "R_Potentiometer_US" (at 55.88 36.83 90)
+      (effects (font (size 1.27 1.27)))
+    )
+    (property "Footprint" "Potentiometer_THT:Potentiometer_Bourns_PTA4543_Single_Slide" (at 55.88 30.48 0)
+      (effects (font (size 1.27 1.27)) hide)
+    )
+    (property "Datasheet" "~" (at 55.88 30.48 0)
+      (effects (font (size 1.27 1.27)) hide)
+    )
+    (pin "1")
+    (pin "2")
+    (pin "3")
+    (instances
+      (project "5431-ButtonBoardButBetter"
+        (path "/85ad268b-acfd-4dd1-a78b-2229ab217983"
+          (reference "RV1") (unit 1)
+        )
+      )

Commit message: added IC footprint-ish
Parts:
- U2: footprint (none) -> Socket:DIP_Socket-16_W4.3_W5.08_W7.62_W10.16_W10.9_3M_216-3340-00-0602J
Changed lines of the file:
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@@
       (effects (font (size 1.27 1.27)) (justify left))
     )
-    (property "Footprint" "" (at 127 29.21 0)
+    (property "Footprint" "Socket:DIP_Socket-16_W4.3_W5.08_W7.62_W10.16_W10.9_3M_216-3340-00-0602J" (at 127 29.21 0)
       (effects (font (size 1.27 1.27)) hide)
     )
