File: ButtonBoard2023.kicad_pcb (KiCad board)
At the start: 2 copper layers, 238.1 x 84.3 mm, 21 parts, among them SW1 SW_DIP_x01, SW10 SW_DIP_x01, SW11 SW_DIP_x01, SW12 SW_DIP_x01, SW13 SW_DIP_x01, SW14 SW_DIP_x01, SW15 SW_DIP_x01, SW16 SW_DIP_x01, SW17 SW_DIP_x01, SW2 SW_DIP_x01, SW3 SW_DIP_x01, SW5 SW_DIP_x01, SW6 SW_DIP_x01, SW7 SW_DIP_x01, SW8 SW_DIP_x01, U1 Pico, U2 MCP3008, U3 COM-09032, U4 COM-09032

Commit message: Everything is project assets, hopefully
Parts:
- removed RV1, RV2: R_Potentiometer_US, Potentiometer_THT:Potentiometer_Bourns_PTA4543_Single_Slide
- removed SW1, SW10, SW11, SW12, SW13, SW14, SW15, SW16, SW2, SW3, SW5, SW6, SW7, SW8: SW_DIP_x01, Button_Switch_Keyboard:SW_Cherry_MX_1.00u_PCB
- removed SW17: SW_DIP_x01, Button_Switch_THT:SW_PUSH_6mm
- removed U1: Pico, MCU_RaspberryPi_and_Boards:RPi_Pico_SMD_TH
- removed U2: MCP3008, Package_DIP:DIP-16_W7.62mm_Socket
- removed U3, U4: COM-09032, COM-09032:XDCR_COM-09032
Other:
- board outline removed

Commit message: ported footprints into schematic
will grab design off my laptop and commit it soon
Parts:
- added RV1: R_Potentiometer_US, Linear Pot:TRIM_PTA4543-2015DPB103, F.Cu at (155.7, 43.6)
- added RV2: R_Potentiometer_US, Linear Pot:TRIM_PTA4543-2015DPB103, F.Cu at (155.7, 56.2)
- added SW1: SW_DIP_x01, KeyboardSwitch:SW_Cherry_MX_1.00u_PCB, F.Cu at (75.9, 42.3)
- added SW10: SW_DIP_x01, KeyboardSwitch:SW_Cherry_MX_1.00u_PCB, F.Cu at (96.1, 82.7)
- added SW11: SW_DIP_x01, KeyboardSwitch:SW_Cherry_MX_1.00u_PCB, F.Cu at (96.1, 102.9)
- added SW12: SW_DIP_x01, KeyboardSwitch:SW_Cherry_MX_1.00u_PCB, F.Cu at (96.1, 123.1)
- added SW13: SW_DIP_x01, KeyboardSwitch:SW_Cherry_MX_1.00u_PCB, F.Cu at (116.3, 42.3)
- added SW14: SW_DIP_x01, KeyboardSwitch:SW_Cherry_MX_1.00u_PCB, F.Cu at (116.3, 62.5)
- added SW15: SW_DIP_x01, KeyboardSwitch:SW_Cherry_MX_1.00u_PCB, F.Cu at (116.3, 82.7)
- added SW16: SW_DIP_x01, KeyboardSwitch:SW_Cherry_MX_1.00u_PCB, F.Cu at (116.3, 102.9)
- added SW17: SW_DIP_x01, Button_Switch_THT:SW_PUSH_6mm, F.Cu at (160.8, 93.6)
- added SW2: SW_DIP_x01, KeyboardSwitch:SW_Cherry_MX_1.00u_PCB, F.Cu at (75.9, 62.5)
- added SW3: SW_DIP_x01, KeyboardSwitch:SW_Cherry_MX_1.00u_PCB, F.Cu at (75.9, 82.7)
- added SW5: SW_DIP_x01, KeyboardSwitch:SW_Cherry_MX_1.00u_PCB, F.Cu at (75.9, 102.9)
- added SW6: SW_DIP_x01, KeyboardSwitch:SW_Cherry_MX_1.00u_PCB, F.Cu at (75.9, 123.1)
- added SW7: SW_DIP_x01, KeyboardSwitch:SW_Cherry_MX_1.00u_PCB, F.Cu at (96.1, 42.3)
- added SW8: SW_DIP_x01, KeyboardSwitch:SW_Cherry_MX_1.00u_PCB, F.Cu at (96.1, 62.5)
- added U1: Pico, MCU_RaspberryPi_and_Boards:RPi_Pico_SMD_TH, F.Cu at (135.9, 118.1)
- added U2: MCP3008, Package_DIP:DIP-16_W7.62mm, F.Cu at (149.6, 93.6)
- added U3: COM-09032, Joystick:XDCR_COM-09032, F.Cu at (138.0, 77.6)
- added U4: COM-09032, Joystick:XDCR_COM-09032, F.Cu at (166.1, 77.6)
