File: ButtonBoard2023.kicad_sch (KiCad schematic)
At the start: 25 parts, among them SW1 SW_DIP_x01, SW10 SW_DIP_x01, SW11 SW_DIP_x01, SW12 SW_DIP_x01, SW13 SW_DIP_x01, SW14 SW_DIP_x01, SW15 SW_DIP_x01, SW16 SW_DIP_x01, SW17 SW_DIP_x01, SW2 SW_DIP_x01, SW3 SW_DIP_x01, SW5 SW_DIP_x01, SW6 SW_DIP_x01, SW7 SW_DIP_x01, SW8 SW_DIP_x01, U1 Pico, U2 MCP3008, U3 COM-09032, U4 COM-09032

Commit message: Everything is project assets, hopefully
Parts:
- RV1, RV2: footprint Potentiometer_THT:Potentiometer_Bourns_PTA4543_Single_Slide -> Linear Pot:TRIM_PTA4543-2015DPB103
- SW1, SW10, SW11, SW12, SW13, SW14, SW15, SW16, SW2, SW3, SW5, SW6, SW7, SW8: footprint Button_Switch_Keyboard:SW_Cherry_MX_1.00u_PCB -> KeyboardSwitch:SW_Cherry_MX_1.00u_PCB
- U2: footprint Package_DIP:DIP-16_W7.62mm_Socket -> Package_DIP:DIP-16_W7.62mm
- U3, U4: footprint COM-09032:XDCR_COM-09032 -> Joystick:XDCR_COM-09032
